File: CH572-LowBOM/CH572-LowBOM.kicad_sch (KiCad schematic)
At the start: 0 parts

Commit message: small works making sure everything going green
none
Parts:
- added J1: USB_A_PCB_Edge_receptacle, Connector_USB_PCB_Edge:USB_A_PCB_Edge_receptacle, symbol Connector_USB_PCB_Edge:USB_A_PCB_Edge_receptacle
- added U1: ~, Ch572D:CH572D, symbol CH572D:CH572D
- added U2: TCR2EF33_LMCT, SOT-25 SMV_TOS, symbol voltage regulator:TCR2EF33_LMCT
- added Y1: XRCGB32M000F2P01R0, XRCGB32M000F2P01R0:OSC_XRCGB32M000F2P01R0, symbol 32mhz crystal:XRCGB32M000F2P01R0
Connections:
- new net: U1.2 (XO), Y1.1
- new net: U1.3 (XI), Y1.3
- new net 5v: J1.1 (VBUS)
- new net D+: J1.3 (D+)
- new net D-: J1.2 (D-)
- new net gnd: J1.4 (GND)
Changed lines of the file:
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@@
 	(generator_version "9.0")
 	(paper "A4")
-	(sheet_instances
-		(path "/"
-			(page "1")
-		)
-	)
-	(embedded_fonts no)
-)

Commit message: nearly just got it done
looks kinda goofy, but real small and decent enough example
Parts:
- added C1, C2: C_0603, Footprint:0603, symbol fab:C_0603
- added C6: 2.2uF, Footprint:0603, symbol 0603:C_0603
- added C7: 0.1uF, Footprint:0603, symbol 0603:C_0603
- added D1, D2: PWRLED, Footprint:LED_1206, symbol fab:LED_1206
- added E2: 2.4ghz, Footprint:antenna, symbol ceramic antenna:AMCA31-2R450G-S1F-T3
- added J2: PinHeader_01x06_P2.54mm_Horizontal_SMD, Footprint:PinHeader_01x06_P2.54mm_Horizontal_SMD, symbol fab:PinHeader_01x06_P2.54mm_Horizontal_SMD
- added R3: 1.5k, Footprint:0603, symbol 0603:R_0603
- added R4, R5: 330, Footprint:0603, symbol 0603:R_0603
- added S1, S2: TL3365AF180QG, Footprint:button, symbol button:TL3365AF180QG
- J1: footprint Connector_USB_PCB_Edge:USB_A_PCB_Edge_receptacle -> Footprint:USB_A_PCB_Edge_receptacle
- U1: footprint Ch572D:CH572D -> Footprint:CH572D
- U2: footprint SOT-25 SMV_TOS -> Footprint:voltage regulator
- Y1: footprint XRCGB32M000F2P01R0:OSC_XRCGB32M000F2P01R0 -> Footprint:32mhz crystal
Connections:
- net 5v is gone; now on net PWR_5V: J1.1 (VBUS)
- net gnd is gone; now on net PWR_GND: J1.4 (GND)
- net D+: now also U1.12 (PA1/UDP/R3/T2/SDA1), R3.2
- net D-: now also U1.11 (PA0/UDM/R2/T3/SCL1)
- net RST: now reaches U1.10 (PA8/SCL/T5/PWM5/RST)
- net RST: now also S2.3, S2.4
- net PA4: now reaches U1.13 (PA4/SCS/PWM4/TMR2)
- net PA4: now also J2.5 (Pin_5)
- net PA5: now reaches U1.14 (PA5/SCK/SCL3)
- net PA5: now also J2.4 (Pin_4)
- net PA6: now reaches U1.15 (PA6/MISO/R4/SDA3)
- net PA6: now also J2.3 (Pin_3)
- net PA7: now reaches U1.16 (PA7/MOSI/T4/PWM1/TMR/RST_/CP1)
- net PA7: now also J2.2 (Pin_2)
- net PA10: now reaches U1.17 (PA10/R6/T7)
- net PA10: now also D2.2 (A)
- net PWR_GND: now reaches U1.21 (GND/EPAD)
- net PWR_GND: now also U2.2 (GND), C1.2, C2.2, J2.6 (Pin_6), R4.1, R5.1, S2.1, S2.2
- net at U1.5 (ANT): now also E2.1
- net PWR_3V3: now reaches U1.6 (VDD33)
- net PWR_3V3: now also U1.7 (VIO33), C6.1, C7.1, D1.2 (A), J2.1 (Pin_1)
- net PWR_5V: now reaches U1.8 (V5)
- net PWR_5V: now also U2.3 (CONTROL)
- net at U2.1 (VIN): now also C2.1
- net at U2.5 (VOUT): now also C1.1
- new net: C6.2, C7.2
- new net: D2.1 (K), R4.2
- new net: R3.1, S1.3, S1.4
- new net: D1.1 (K), R5.2
- new net +3.3V: S1.1, S1.2
Other:
- moved on the sheet: J1, U1, U2, Y1

Commit message: work done kinda needs a bit more
Connections:
- net PA10: no longer U1.17 (PA10/R6/T7)
- net PWR_GND: now also C6.2, C7.2
- net PA9: now reaches U1.9 (PA9/SDA/R5/TMR3)
