File: CH572-LowBOM/CH572-LowBOM.kicad_pcb (KiCad board)
At the start: 2 copper layers, 12 x 14 mm, 17 parts, among them J1 USB_A_PCB_Edge_receptacle, J2 PinHeader_01x06_P2.54mm_Horiz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, U2 TCR2EF33_LMCT, Y1 XRCGB32M000F2P01R0

Commit message: work done kinda needs a bit more
Parts:
- moved U1 38.6 mm to (104.9, 148.8), turned to 180 degrees
- moved J1 31.1 mm to (89.7, 150.8), turned to 0 degrees
- moved C7 19.7 mm to (95.2, 123.3), turned to -150 degrees
- moved C6 18.8 mm to (95.9, 124.5), turned to -150 degrees
- moved R3 18.4 mm to (116.6, 130.6), turned to 180 degrees
- moved R4 13.1 mm to (107.3, 127.2), turned to -90 degrees
- moved D1 12.4 mm to (111.7, 130.0), turned to 180 degrees
- moved Y1 11.7 mm to (113.8, 119.1), turned to 30 degrees
- moved S1 11.6 mm to (120.2, 128.7)
- moved S2 10.5 mm to (103.9, 128.8)
- moved D2 9.88 mm to (111.7, 127.8), turned to 0 degrees
- moved R5 9.52 mm to (115.9, 127.2), turned to -90 degrees
- moved C1 6.90 mm to (106.8, 120.3)
- moved C2 6.90 mm to (103.4, 117.9)
- moved U2 6.90 mm to (103.9, 120.3)
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Connections:
- C6 pad 2: Net-(C6-Pad2) -> PWR_GND
- C7 pad 2: Net-(C6-Pad2) -> PWR_GND
- U1 pad 17: PA10 -> unconnected-(U1-PA10/R6/T7-Pad17)
- U1 pad 9: unconnected-(U1-PA9/SDA/R5/TMR3-Pad9) -> PA9
Other:
- board size 12 x 14 mm -> 14 x 12 mm

Commit message: work
Parts:
- J1: moved to B.Cu
- moved J2 52.6 mm to (130.3, 162.1), turned to -90 degrees
- moved E2 42.0 mm to (121.5, 139.5)
- moved Y1 37.4 mm to (112.1, 156.5), turned to 180 degrees
- moved S1 32.5 mm to (101.5, 155.3), turned to 180 degrees
- moved C1 31.7 mm to (103.8, 151.9)
- moved U2 31.6 mm to (100.8, 151.7)
- moved C2 31.6 mm to (103.5, 149.5)
- moved C7 28.6 mm to (106.7, 149.5), turned to 180 degrees
- moved R3 26.5 mm to (107.5, 155.4), turned to 90 degrees
- moved C6 26.3 mm to (107.5, 148.1), turned to 180 degrees
- moved R5 25.8 mm to (106.1, 151.1), turned to 0 degrees
- moved D1 25.1 mm to (105.7, 154.4), turned to -90 degrees
- moved R4 19.8 mm to (105.2, 146.9), turned to 90 degrees
- moved D2 18.8 mm to (108.6, 146.3)
- moved S2 18.3 mm to (101.5, 146.9), turned to 180 degrees
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Routing:
- net Net-(U2-VIN): track 1.58 -> 0.00 mm
- net Net-(U2-VOUT): track 1.57 -> 0.00 mm

Commit message: final of the night
Parts:
- moved E2 12.4 mm to (113.0, 148.4)
- moved J2 9.79 mm to (127.8, 152.6)
- moved R5 4.69 mm to (105.5, 155.7), turned to -90 degrees
- moved C2 4.15 mm to (99.6, 150.8), turned to -90 degrees
- moved D1 3.91 mm to (108.9, 156.6), turned to 0 degrees
- moved C6 3.82 mm to (111.1, 146.7), turned to 0 degrees
- moved C7 3.03 mm to (107.9, 146.7)
- moved Y1 2.88 mm to (112.3, 153.6), turned to 0 degrees
- moved U2 1.86 mm to (102.4, 150.8)
- moved C1 1.72 mm to (105.2, 150.8)
- moved R4 1.48 mm to (105.6, 145.5)
- moved D2 1.48 mm to (109.0, 144.9)
- moved S2 1.46 mm to (101.9, 145.6)
- moved U1 1.36 mm to (109.7, 148.2)
- moved R3 0.97 mm to (108.0, 154.7), turned to 0 degrees
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Connections:
- C1 pad 1: Net-(U2-VOUT) -> PWR_3V3
- C2 pad 1: Net-(U2-VIN) -> PWR_5V
- D2 pad 2: PA10 -> PA9
- J2 pad 2: PA7 -> PA10
- J2 pad 3: PA6 -> PA11
- J2 pad 4: PA5 -> PA2
- J2 pad 5: PA4 -> PA3
- S1 pad 1: +3.3V -> PWR_3V3
- S1 pad 2: +3.3V -> PWR_3V3
- U1 pad 1: unconnected-(U1-PA3/T/R1/SCL2/SCK_/PWM3/CP0-Pad1) -> PA3
- U1 pad 13: PA4 -> unconnected-(U1-PA4/SCS/PWM4/TMR2-Pad13)
- U1 pad 14: PA5 -> unconnected-(U1-PA5/SCK/SCL3-Pad14)
- U1 pad 15: PA6 -> unconnected-(U1-PA6/MISO/R4/SDA3-Pad15)
- U1 pad 16: PA7 -> unconnected-(U1-PA7/MOSI/T4/PWM1/TMR/RST_/CP1-Pad16)
- U1 pad 17: unconnected-(U1-PA10/R6/T7-Pad17) -> PA10
- U1 pad 18: unconnected-(U1-PA11/R7/T6-Pad18) -> PA11
- U1 pad 20: unconnected-(U1-PA2/R/T1/SDA2/SCS_/PWM2/TMR1/CN-Pad20) -> PA2
- U2 pad 1: Net-(U2-VIN) -> PWR_5V
- U2 pad 5: Net-(U2-VOUT) -> PWR_3V3
Routing:
- net PWR_3V3: track 0.00 -> 49.3 mm, vias 0 -> 2
- net D+: track 0.00 -> 24.3 mm, vias 0 -> 1
- net PWR_5V: track 0.00 -> 23.7 mm, vias 0 -> 1
- net PA10: track 0.00 -> 20.6 mm, vias 0 -> 2
- net D-: track 0.00 -> 19.7 mm, vias 0 -> 1
- net PA11: track 0.00 -> 17.2 mm
- net Net-(R3-Pad1): track 0.00 -> 16.8 mm
- net PA2: track 0.00 -> 13.7 mm
- net RST: track 0.00 -> 10.7 mm, vias 0 -> 2
- net PA3: track 0.00 -> 9.34 mm, vias 0 -> 2
- net PWR_GND: track 0.00 -> 8.27 mm, vias 0 -> 35
- net Net-(U1-XI): track 0.00 -> 5.40 mm
- net PA9: track 0.00 -> 4.67 mm, vias 0 -> 2
- net Net-(U1-ANT): track 0.00 -> 3.99 mm
- net Net-(U1-XO): track 0.00 -> 3.81 mm
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- added copper zone on B.Cu, net PWR_GND
Other:
- board size 14 x 12 mm -> 45.7 x 15.5 mm
